File: hardware/ESP32S3_RF_DevBoard.kicad_pcb (KiCad board)
At the start: 4 copper layers, 25.4 x 60 mm, 37 parts, among them J1 USB4105-GF-A, J2 Conn_01x22, J3 Conn_01x22, SW1 BOOT, SW2 RESET, U1 ESD122DMYR, U2 LD1117DT33CTR, U3 ESP32-S3-WROOM-1-N8, U4 SN74AHCT1G125DBVR

Commit message: - working on the diff pairs (D-/D+) of USB.
Parts:
- moved R6 1.65 mm to (143.9, 90.1)
- moved R7 1.65 mm to (145.4, 90.1)
Changed lines of the file:
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@@
 	(footprint "Resistor_SMD:R_0603_1608Metric"
 		(layer "F.Cu")
-		(at 145.5 89.675 -90)
+		(at 143.9 90.075 -90)
 		(descr "Resistor SMD 0603 (1608 Metric), square (rectangular) end terminal, IPC-7351 nominal, (Body size source: IPC-SM-782 page 72, https://www.pcb-3d.com/wordpress/wp-content/uploads/ipc-sm-782a_amendment_1_and_2.pdf)")
 		(tags "resistor")
 		(property "Reference" "R6"
-			(at 0 1.5 90)
+			(at 2.05 0.05 180)
 			(layer "F.SilkS")
 			(effects
@@
 	(footprint "Resistor_SMD:R_0603_1608Metric"
 		(layer "F.Cu")
-		(at 147 89.675 -90)
+		(at 145.4 90.075 -90)
 		(descr "Resistor SMD 0603 (1608 Metric), square (rectangular) end terminal, IPC-7351 nominal, (Body size source: IPC-SM-782 page 72, https://www.pcb-3d.com/wordpress/wp-content/uploads/ipc-sm-782a_amendment_1_and_2.pdf)")
 		(tags "resistor")
 		(property "Reference" "R7"
-			(at 0 -1.43 90)
-			(layer "F.SilkS")
-			(effects
+			(at 2.1 -0.15 180)
+			(layer "F.SilkS")
+			(effects

Commit message: working on routing still - completed USB routing diff pair
Parts:
- moved R6 1.33 mm to (144.8, 91.1)
- moved R7 1.33 mm to (146.2, 91.1)
- moved TP1 1.27 mm to (144.8, 122.8)
- moved U1 0.84 mm to (154.7, 118.1)
- moved R9 0.74 mm to (149.5, 113.8)
- moved SW2 0.74 mm to (146.4, 118.2)
- moved TP4 0.74 mm to (149.5, 116.8)
- moved TP5 0.74 mm to (149.4, 110.3)
- moved SW1 0.74 mm to (146.4, 112.4)
- moved R10 0.30 mm to (159.1, 114.2)
- moved U4 0.25 mm to (158.8, 111.8)
- moved C7 0.25 mm to (161.6, 111.8)
- moved R8 0.25 mm to (156.1, 111.6)
Routing:
- net /USB_D-: track 0.00 -> 36.4 mm, vias 0 -> 2
- net /USB_D+: track 0.00 -> 34.1 mm
- net /+5V_USB: track 0.00 -> 32.8 mm
- net /USB_ESP_D-: track 0.00 -> 7.42 mm
- net /USB_ESP_D+: track 0.00 -> 5.59 mm
- net GND: track 0.00 -> 3.69 mm, vias 7 -> 9
- added copper zone on In2.Cu, net GND

Commit message: - 5 unconnected components as of now! - trying to route the rest of the GPIO and CHIP_PU traces - will deal with silkscreen and footprint warnings last !
Parts:
- R4: moved to F.Cu
- TP6, TP7: moved to B.Cu
- moved TP7 24.3 mm to (159.0, 74.2), turned to 180 degrees
- moved R4 21.6 mm to (150.8, 91.5), turned to 180 degrees
- moved TP6 18.6 mm to (159.0, 78.0), turned to 180 degrees
- moved D2 10.00 mm to (148.4, 96.7), turned to -90 degrees
- moved R3 8.72 mm to (150.0, 96.8), turned to -90 degrees
- moved R10 4.00 mm to (160.5, 110.5), turned to 90 degrees
- moved C5 3.23 mm to (150.0, 70.8)
- moved LED1 2.59 mm to (157.4, 114.0)
- moved C7 2.11 mm to (160.8, 113.8), turned to 0 degrees
- moved TP2 2.02 mm to (159.0, 90.8)
- moved TP3 1.63 mm to (159.6, 93.9)
- moved U4 0.90 mm to (158.2, 111.0), turned to 90 degrees
- moved TP5 0.57 mm to (149.4, 110.9)
- moved R8 0.48 mm to (155.8, 111.2)
- moved R5 0.26 mm to (146.5, 73.2)
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Connections:
- J2 pad 3: /CHIP_PU -> /GPIO4
- J2 pad 4: /GPIO4 -> /CHIP_PU
- J3 pad 10: /GPIO38 -> /GPIO37
- J3 pad 11: /GPIO37 -> /GPIO38
- J3 pad 19: /USB_ESP_D+ -> unconnected-(J3-Pin_19-Pad19)
- J3 pad 2: /TX -> /GPIO1
- J3 pad 20: /USB_ESP_D- -> unconnected-(J3-Pin_20-Pad20)
- J3 pad 3: /RX -> /GPIO2
- J3 pad 4: /GPIO1 -> /TX
- J3 pad 5: /GPIO2 -> /RX
Routing:
- net /ESP_3V3: track 0.00 -> 57.6 mm, vias 0 -> 3
- net /GPIO0: track 0.00 -> 52.2 mm, vias 0 -> 3
- net /CHIP_PU: track 0.00 -> 50.5 mm, vias 0 -> 3
- net /+3V3: track 0.00 -> 48.7 mm, vias 0 -> 2
- net /GPIO14: track 0.00 -> 40.9 mm, vias 0 -> 1
- net /GPIO13: track 0.00 -> 38.3 mm, vias 0 -> 1
- net /GPIO38: track 0.00 -> 37.3 mm, vias 0 -> 2
- net /GPIO12: track 0.00 -> 35.4 mm, vias 0 -> 1
- net /GPIO21: track 0.00 -> 31.4 mm, vias 0 -> 1
- net /GPIO10: track 0.00 -> 31.1 mm, vias 0 -> 1
- net /GPIO11: track 0.00 -> 31.0 mm, vias 0 -> 1
- net /GPIO47: track 0.00 -> 27.8 mm, vias 0 -> 1
- net /GPIO48: track 0.00 -> 24.8 mm, vias 0 -> 1
- net GND: track 3.69 -> 28.5 mm, vias 9 -> 26
- net /GPIO9: track 0.00 -> 24.6 mm, vias 0 -> 1
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- added copper zone on F.Cu, net /+3V3

Commit message: working on silkscreen warnings and fixing . - all routing complete (0 unconnections) - verfiy in JLCPCB USB NPTH hole placeement (may have to exclude the error if JLCPCB clears through dfm)
Parts:
- removed TP6, TP7: TestPoint, TestPoint:TestPoint_Pad_D1.0mm
- moved TP5 0.11 mm to (149.4, 110.8)
Routing:
- net /+5V_USB: track 43.8 -> 60.7 mm, vias 0 -> 2
- net /CHIP_PU: track 50.5 -> 62.2 mm
- net /GPIO42: track 0.00 -> 11.1 mm, vias 0 -> 1
- net /TX: track 15.3 -> 7.32 mm
- net /RX: track 12.4 -> 8.39 mm, vias 1 -> 0
- net /GPIO38: track 37.3 -> 39.2 mm
- net /GPIO37: track 14.2 -> 15.3 mm
- net /GPIO0: track 52.2 -> 51.7 mm
- added copper zone on In2.Cu, net /+3V3
Other:
- board text removed: "RX"
- board text removed: "TX"
